File: Volets/Volets.kicad_sch (KiCad schematic)
At the start: 0 parts

Commit message: Mise à jour
Parts:
- added U1: LM75B, symbol Sensor_Temperature:LM75B
- added U2: TCS3200, TCS3200:SOIC127P600X175-8N, symbol TCS3200:TCS3200
Other:
- note added: "Capteur température"
- note added: "capteur lumière"

Commit message: Mise à jour
Parts:
- added C1: 0.1uF, symbol Device:C
- added C2: 0.1-0.01nF, symbol Device:C
- added D1, D2, D3, D4: LED, symbol Device:LED
- added J1: Conn_01x03, symbol Connector_Generic:Conn_01x03
- added J2: Conn_01x02, symbol Connector_Generic:Conn_01x02
- added J3, J4: Conn_01x04, symbol Connector_Generic:Conn_01x04
- added R1, R2, R5, R6: 10k, symbol Device:R
- added R10, R7, R8, R9: R, symbol Device:R
- added R3: 200k, symbol Device:R
- added R4: 1k, symbol Device:R
Connections:
- net S0: now reaches U2.1 (S0)
- net S0: now also J3.1 (Pin_1), R5.2
- net S1: now reaches U2.2 (S1)
- net S1: now also J3.2 (Pin_2), R6.2
- net OE: now reaches U2.3 (~{OE})
- net OE: now also J3.3 (Pin_3)
- net GND: now reaches U2.4 (GND)
- net GND: now also U1.4 (GND), C1.1, C2.2, J3.4 (Pin_4), R10.2, R7.2, R8.2, R9.2
- net Vcc: now reaches U2.5 (VDD)
- net Vcc: now also C2.1, D1.2 (A), D2.2 (A), D3.2 (A), D4.2 (A), J4.4 (Pin_4), R5.1, R6.1
- net at U2.6 (OUT): now also R4.1
- net S2: now reaches U2.7 (S2)
- net S2: now also J4.1 (Pin_1)
- net S3: now reaches U2.8 (S3)
- net S3: now also J4.2 (Pin_2)
- net I2C: now reaches U1.1 (SDA)
- net I2C: now also J2.1 (Pin_1), R2.2
- net BUS: now reaches U1.2 (SCL)
- net BUS: now also J2.2 (Pin_2), R1.2
- net at U1.3 (O.S.): now also R3.2
- net A2: now reaches U1.5 (A2)
- net A2: now also J1.3 (Pin_3)
- net A1: now reaches U1.6 (A1)
- net A1: now also J1.2 (Pin_2)
- net A0: now reaches U1.7 (A0)
- net A0: now also J1.1 (Pin_1)
- net +5V: now reaches U1.8 (+Vs)
- net +5V: now also C1.2, R1.1, R2.1, R3.1
- new net: D2.1 (K), R8.1
- new net: D3.1 (K), R9.1
- new net: D1.1 (K), R7.1
- new net: D4.1 (K), R10.1
- new net out: J4.3 (Pin_3), R4.2
Other:
- note added: "connecteur"
- moved on the sheet: U1
